Commit message: Standardize robot naming to tiangong3

File: source/whole_body_tracking/whole_body_tracking/assets/tiangong3/urdf/tiangong3.urdf (robot description, URDF)
Before this commit: robot tiangong2dex_urdf, 39 links, 38 joints
Links:
- link ankle_pitch_l_link: geometry visual mesh filename=../meshes_new/ankle_pitch_l_link.STL
- link ankle_pitch_r_link: geometry visual mesh filename=../meshes_new/ankle_pitch_r_link.STL
- link ankle_roll_l_link: geometry collision cylinder length=0.06 radius=0.012; collision cylinder length=0.06 radius=0.012
- link ankle_roll_r_link: geometry collision cylinder length=0.06 radius=0.012; collision cylinder length=0.06 radius=0.012
- link camera_body_front_link: geometry visual mesh filename=../meshes_new/camera_body_front_link.STL
- link camera_head_link: geometry visual mesh filename=../meshes_new/camera_head_link.STL
- link elbow_pitch_l_link: geometry visual mesh filename=../meshes_new/elbow_pitch_l_link.STL
- link elbow_pitch_r_link: geometry visual mesh filename=../meshes_new/elbow_pitch_r_link.STL
- link elbow_yaw_l_link: geometry visual mesh filename=../meshes_new/elbow_yaw_l_link.STL
- link elbow_yaw_r_link: geometry visual mesh filename=../meshes_new/elbow_yaw_r_link.STL
- link head_pitch_link: geometry visual mesh filename=../meshes_new/head_pitch_link.STL
- link head_yaw_link: geometry visual mesh filename=../meshes_new/head_yaw_link.STL
- link hip_pitch_l_link: geometry collision cylinder length=0.07 radius=0.06; visual mesh filename=../meshes_new/hip_pitch_l_link.STL
- link hip_pitch_r_link: geometry collision cylinder length=0.07 radius=0.06; visual mesh filename=../meshes_new/hip_pitch_r_link.STL
- link hip_roll_l_link: geometry visual mesh filename=../meshes_new/hip_roll_l_link.STL
- link hip_roll_r_link: geometry visual mesh filename=../meshes_new/hip_roll_r_link.STL
- link hip_yaw_l_link: geometry collision mesh filename=../meshes_new/hip_yaw_l_link.STL; visual mesh filename=../meshes_new/hip_yaw_l_link.STL
- link hip_yaw_r_link: geometry collision mesh filename=../meshes_new/hip_yaw_r_link.STL; visual mesh filename=../meshes_new/hip_yaw_r_link.STL
- link imu_head_link: geometry visual mesh filename=../meshes_new/imu_head_link.STL
- link imu_waist_link: geometry visual mesh filename=../meshes_new/imu_waist_link.STL
- link knee_pitch_l_link: geometry collision mesh filename=../meshes_new/knee_pitch_l_link.STL; visual mesh filename=../meshes_new/knee_pitch_l_link.STL
- link knee_pitch_r_link: geometry collision mesh filename=../meshes_new/knee_pitch_r_link.STL; visual mesh filename=../meshes_new/knee_pitch_r_link.STL
- link left_tcp_link: geometry collision mesh filename=../meshes_new/left_tcp_link.STL; visual mesh filename=../meshes_new/left_tcp_link.STL
- link pelvis: geometry collision mesh filename=../meshes_new/pelvis.STL; visual mesh filename=../meshes_new/pelvis.STL
- link radar_head_link: geometry visual mesh filename=../meshes_new/radar_head_link.STL
- link right_tcp_link: geometry collision mesh filename=../meshes_new/right_tcp_link.STL; visual mesh filename=../meshes_new/right_tcp_link.STL
- link shoulder_pitch_l_link: geometry visual mesh filename=../meshes_new/shoulder_pitch_l_link.STL
- link shoulder_pitch_r_link: geometry visual mesh filename=../meshes_new/shoulder_pitch_r_link.STL
- link shoulder_roll_l_link: geometry visual mesh filename=../meshes_new/shoulder_roll_l_link.STL
- link shoulder_roll_r_link: geometry visual mesh filename=../meshes_new/shoulder_roll_r_link.STL
- link shoulder_yaw_l_link: geometry collision mesh filename=../meshes_new/shoulder_yaw_l_link.STL; visual mesh filename=../meshes_new/shoulder_yaw_l_link.STL
- link shoulder_yaw_r_link: geometry collision mesh filename=../meshes_new/shoulder_yaw_r_link.STL; visual mesh filename=../meshes_new/shoulder_yaw_r_link.STL
- link waist_pitch_link: geometry collision mesh filename=../meshes_new/waist_pitch_link.STL; visual mesh filename=../meshes_new/waist_pitch_link.STL
- link waist_roll_link: geometry visual mesh filename=../meshes_new/waist_roll_link.STL
- link waist_yaw_link: geometry visual mesh filename=../meshes_new/waist_yaw_link.STL
- link wrist_pitch_l_link: geometry collision mesh filename=../meshes_new/wrist_pitch_l_link.STL; visual mesh filename=../meshes_new/wrist_pitch_l_link.STL
- link wrist_pitch_r_link: geometry collision mesh filename=../meshes_new/wrist_pitch_r_link.STL; visual mesh filename=../meshes_new/wrist_pitch_r_link.STL
- link wrist_roll_l_link: geometry visual mesh filename=../meshes_new/wrist_roll_l_link.STL
- link wrist_roll_r_link: geometry visual mesh filename=../meshes_new/wrist_roll_r_link.STL
Joints:
- joint elbow_yaw_l_joint: type revolute -> fixed
- joint elbow_yaw_r_joint: type revolute -> fixed
- joint head_pitch_joint: type revolute -> fixed
- joint head_yaw_joint: type revolute -> fixed
- joint wrist_pitch_l_joint: type revolute -> fixed
- joint wrist_pitch_r_joint: type revolute -> fixed
- joint wrist_roll_l_joint: type revolute -> fixed
- joint wrist_roll_r_joint: type revolute -> fixed

File: source/whole_body_tracking/whole_body_tracking/assets/tiangong3/urdf/tiangong3.urdf.xacro (robot description, xacro)
@@ -1,4 +1,4 @@
 <?xml version='1.0' encoding='utf-8'?>
-<robot name="tiangong2dex_urdf">
+<robot name="tiangong3_urdf" xmlns:xacro="http://wiki.ros.org/xacro">
   <link name="pelvis">
     <inertial>
@@ -10,5 +10,5 @@
       <origin xyz="0 0 0" rpy="0 0 0" />
       <geometry>
-        <mesh filename="../meshes_new/pelvis.STL" />
+        <mesh filename="package://tiangong3_urdf/meshes/pelvis.STL" />
       </geometry>
       <material name="pelvis_color">
@@ -19,5 +19,5 @@
       <origin xyz="0 0 0" rpy="0 0 0" />
       <geometry>
-        <mesh filename="../meshes_new/pelvis.STL" />
+        <mesh filename="package://tiangong3_urdf/meshes/pelvis.STL" />
       </geometry>
     </collision>
@@ -32,20 +32,14 @@
       <origin xyz="0 0 0" rpy="0 0 0" />
       <geometry>
-        <mesh filename="../meshes_new/hip_pitch_l_link.STL" />
-      </geometry>
-      <material name="">
-        <color rgba="0.752941176470588 0.752941176470588 0.752941176470588 1" />
-      </material>
-    </visual>
-    <!-- <collision>
-      <origin xyz="0 0 0" rpy="0 0 0" />
-      <geometry>
-        <mesh filename="../meshes_new/hip_pitch_l_link.STL" />
-      </geometry>
-    </collision> -->
-    <collision>
-      <origin xyz="0 0.08 -0.02" rpy="0 1.5708 0"/>
-      <geometry>
-        <cylinder radius="0.06" length="0.07"/>
+        <mesh filename="package://tiangong3_urdf/meshes/hip_pitch_l_link.STL" />
+      </geometry>
+      <material name="">
+        <color rgba="0.752941176470588 0.752941176470588 0.752941176470588 1" />
+      </material>
+    </visual>
+    <collision>
+      <origin xyz="0 0 0" rpy="0 0 0" />
+      <geometry>
+        <mesh filename="package://tiangong3_urdf/meshes/hip_pitch_l_link.STL" />
       </geometry>
     </collision>
@@ -67,22 +61,16 @@
       <origin xyz="0 0 0" rpy="0 0 0" />
       <geometry>
-        <mesh filename="../meshes_new/hip_roll_l_link.STL" />
-      </geometry>
-      <material name="">
-        <color rgba="0.752941176470588 0.752941176470588 0.752941176470588 1" />
-      </material>
-    </visual>
-    <!-- <collision>
-      <origin xyz="0 0 0" rpy="0 0 0" />
-      <geometry>
-        <mesh filename="../meshes_new/hip_roll_l_link.STL" />
-      </geometry>
-    </collision> -->
-    <!-- <collision>
-      <origin xyz="0 0 0" rpy="0 1.57079632679 0" />
-      <geometry>
-        <cylinder radius="0.065" length="0.10" />
-      </geometry>
-    </collision> -->
+        <mesh filename="package://tiangong3_urdf/meshes/hip_roll_l_link.STL" />
+      </geometry>
+      <material name="">
+        <color rgba="0.752941176470588 0.752941176470588 0.752941176470588 1" />
+      </material>
+    </visual>
+    <collision>
+      <origin xyz="0 0 0" rpy="0 0 0" />
+      <geometry>
+        <mesh filename="package://tiangong3_urdf/meshes/hip_roll_l_link.STL" />
+      </geometry>
+    </collision>
   </link>
   <joint name="hip_roll_l_joint" type="revolute">
@@ -102,14 +90,14 @@
       <origin xyz="0 0 0" rpy="0 0 0" />
       <geometry>
-        <mesh filename="../meshes_new/hip_yaw_l_link.STL" />
-      </geometry>
-      <material name="">
-        <color rgba="0.752941176470588 0.752941176470588 0.752941176470588 1" />
-      </material>
-    </visual>
-    <collision>
-      <origin xyz="0 0 0" rpy="0 0 0" />
-      <geometry>
-        <mesh filename="../meshes_new/hip_yaw_l_link.STL" />
+        <mesh filename="package://tiangong3_urdf/meshes/hip_yaw_l_link.STL" />
+      </geometry>
+      <material name="">
+        <color rgba="0.752941176470588 0.752941176470588 0.752941176470588 1" />
+      </material>
+    </visual>
+    <collision>
+      <origin xyz="0 0 0" rpy="0 0 0" />
+      <geometry>
+        <mesh filename="package://tiangong3_urdf/meshes/hip_yaw_l_link.STL" />
       </geometry>
     </collision>
@@ -131,14 +119,14 @@
       <origin xyz="0 0 0" rpy="0 0 0" />
       <geometry>
-        <mesh filename="../meshes_new/knee_pitch_l_link.STL" />
-      </geometry>
-      <material name="">
-        <color rgba="0.752941176470588 0.752941176470588 0.752941176470588 1" />
-      </material>
-    </visual>
-    <collision>
-      <origin xyz="0 0 0" rpy="0 0 0" />
-      <geometry>
-        <mesh filename="../meshes_new/knee_pitch_l_link.STL" />
+        <mesh filename="package://tiangong3_urdf/meshes/knee_pitch_l_link.STL" />
+      </geometry>
+      <material name="">
+        <color rgba="0.752941176470588 0.752941176470588 0.752941176470588 1" />
+      </material>
+    </visual>
+    <collision>
+      <origin xyz="0 0 0" rpy="0 0 0" />
+      <geometry>
+        <mesh filename="package://tiangong3_urdf/meshes/knee_pitch_l_link.STL" />
       </geometry>
     </collision>
@@ -160,16 +148,16 @@
       <origin xyz="0 0 0" rpy="0 0 0" />
       <geometry>
-        <mesh filename="../meshes_new/ankle_pitch_l_link.STL" />
-      </geometry>
-      <material name="">
-        <color rgba="0.752941176470588 0.752941176470588 0.752941176470588 1" />
-      </material>
-    </visual>
-    <!-- <collision>
-      <origin xyz="0 0 0" rpy="0 0 0" />
-      <geometry>
-        <mesh filename="../meshes_new/ankle_pitch_l_link.STL" />
-      </geometry>
-    </collision> -->
+        <mesh filename="package://tiangong3_urdf/meshes/ankle_pitch_l_link.STL" />
+      </geometry>
+      <material name="">
+        <color rgba="0.752941176470588 0.752941176470588 0.752941176470588 1" />
+      </material>
+    </visual>
+    <collision>
+      <origin xyz="0 0 0" rpy="0 0 0" />
+      <geometry>
+        <mesh filename="package://tiangong3_urdf/meshes/ankle_pitch_l_link.STL" />
+      </geometry>
+    </collision>
   </link>
   <joint name="ankle_pitch_l_joint" type="revolute">
@@ -189,56 +177,14 @@
       <origin xyz="0 0 0" rpy="0 0 0" />
       <geometry>
-        <mesh filename="../meshes_new/ankle_roll_l_link.STL" />
-      </geometry>
-      <material name="">
-        <color rgba="0.752941176470588 0.752941176470588 0.752941176470588 1" />
-      </material>
-    </visual>
-    <!-- <collision>
-      <origin xyz="0 0 0" rpy="0 0 0" />
-      <geometry>
-        <mesh filename="../meshes_new/ankle_roll_l_link.STL" />
-      </geometry>
-    </collision> -->
-    <collision name="foot_left_front_outer">
-      <origin xyz="0.085 -0.03 -0.046" rpy="0 1.5708 0" />
-      <geometry>
-        <cylinder radius="0.012" length="0.06" />
-      </geometry>
-    </collision>
-    <collision name="foot_left_front_inner">
-      <origin xyz="0.085 0.03 -0.046" rpy="0 1.5708 0" />
-      <geometry>
-        <cylinder radius="0.012" length="0.06" />
-      </geometry>
-    </collision>
-    <collision name="foot_left_mid_outer">
-      <origin xyz="0.045 -0.02 -0.046" rpy="0 -1.5708 0" />
-      <geometry>
-        <cylinder radius="0.01" length="0.20" />
-      </geometry>
-    </collision>
-    <collision name="foot_left_mid_inner">
-      <origin xyz="0.045 0.02 -0.046" rpy="0 -1.5708 0" />
-      <geometry>
-        <cylinder radius="0.01" length="0.20" />
-      </geometry>
-    </collision>
-    <collision name="foot_left_strip_outer">
-      <origin xyz="0.045 -0.01 -0.046" rpy="0 -1.5708 0" />
-      <geometry>
-        <cylinder radius="0.012" length="0.22" />
-      </geometry>
-    </collision>
-    <collision name="foot_left_strip_center">
-      <origin xyz="0.045 0 -0.046" rpy="0 -1.5708 0" />
-      <geometry>
-        <cylinder radius="0.012" length="0.24" />
-      </geometry>
-    </collision>
-    <collision name="foot_left_strip_inner">
-      <origin xyz="0.045 0.01 -0.046" rpy="0 -1.5708 0" />
-      <geometry>
-        <cylinder radius="0.012" length="0.22" />
+        <mesh filename="package://tiangong3_urdf/meshes/ankle_roll_l_link.STL" />
+      </geometry>
+      <material name="">
+        <color rgba="0.752941176470588 0.752941176470588 0.752941176470588 1" />
+      </material>
+    </visual>
+    <collision>
+      <origin xyz="0 0 0" rpy="0 0 0" />
+      <geometry>
+        <mesh filename="package://tiangong3_urdf/meshes/ankle_roll_l_link.STL" />
       </geometry>
     </collision>
@@ -260,20 +206,14 @@
       <origin xyz="0 0 0" rpy="0 0 0" />
       <geometry>
-        <mesh filename="../meshes_new/hip_pitch_r_link.STL" />
-      </geometry>
-      <material name="">
-        <color rgba="0.752941176470588 0.752941176470588 0.752941176470588 1" />
-      </material>
-    </visual>
-    <!-- <collision>
-      <origin xyz="0 0 0" rpy="0 0 0" />
-      <geometry>
-        <mesh filename="../meshes_new/hip_pitch_r_link.STL" />
-      </geometry>
-    </collision> -->
-    <collision>
-      <origin xyz="0 -0.08 -0.02" rpy="0 1.5708 0"/>
-      <geometry>
-        <cylinder radius="0.06" length="0.07"/>
+        <mesh filename="package://tiangong3_urdf/meshes/hip_pitch_r_link.STL" />
+      </geometry>
+      <material name="">
+        <color rgba="0.752941176470588 0.752941176470588 0.752941176470588 1" />
+      </material>
+    </visual>
+    <collision>
+      <origin xyz="0 0 0" rpy="0 0 0" />
+      <geometry>
+        <mesh filename="package://tiangong3_urdf/meshes/hip_pitch_r_link.STL" />
       </geometry>
     </collision>
@@ -295,22 +235,16 @@
       <origin xyz="0 0 0" rpy="0 0 0" />
       <geometry>
-        <mesh filename="../meshes_new/hip_roll_r_link.STL" />
-      </geometry>
-      <material name="">
-        <color rgba="0.752941176470588 0.752941176470588 0.752941176470588 1" />
-      </material>
-    </visual>
-    <!-- <collision>
-      <origin xyz="0 0 0" rpy="0 0 0" />
-      <geometry>
-        <mesh filename="../meshes_new/hip_roll_r_link.STL" />
-      </geometry>
-    </collision> -->
-    <!-- <collision>
-      <origin xyz="0 0 0" rpy="0 1.57079632679 0" />
-      <geometry>
-        <cylinder radius="0.065" length="0.10" />
-      </geometry>
-    </collision> -->
+        <mesh filename="package://tiangong3_urdf/meshes/hip_roll_r_link.STL" />
+      </geometry>
+      <material name="">
+        <color rgba="0.752941176470588 0.752941176470588 0.752941176470588 1" />
+      </material>
+    </visual>
+    <collision>
+      <origin xyz="0 0 0" rpy="0 0 0" />
+      <geometry>
+        <mesh filename="package://tiangong3_urdf/meshes/hip_roll_r_link.STL" />
+      </geometry>
+    </collision>
   </link>
   <joint name="hip_roll_r_joint" type="revolute">
@@ -330,14 +264,14 @@
       <origin xyz="0 0 0" rpy="0 0 0" />
       <geometry>
-        <mesh filename="../meshes_new/hip_yaw_r_link.STL" />
-      </geometry>
-      <material name="">
-        <color rgba="0.752941176470588 0.752941176470588 0.752941176470588 1" />
-      </material>
-    </visual>
-    <collision>
-      <origin xyz="0 0 0" rpy="0 0 0" />
-      <geometry>
-        <mesh filename="../meshes_new/hip_yaw_r_link.STL" />
+        <mesh filename="package://tiangong3_urdf/meshes/hip_yaw_r_link.STL" />
+      </geometry>
+      <material name="">
+        <color rgba="0.752941176470588 0.752941176470588 0.752941176470588 1" />
+      </material>
+    </visual>
+    <collision>
+      <origin xyz="0 0 0" rpy="0 0 0" />
+      <geometry>
+        <mesh filename="package://tiangong3_urdf/meshes/hip_yaw_r_link.STL" />
       </geometry>
     </collision>
@@ -359,14 +293,14 @@
       <origin xyz="0 0 0" rpy="0 0 0" />
       <geometry>
-        <mesh filename="../meshes_new/knee_pitch_r_link.STL" />
-      </geometry>
-      <material name="">
-        <color rgba="0.752941176470588 0.752941176470588 0.752941176470588 1" />
-      </material>
-    </visual>
-    <collision>
-      <origin xyz="0 0 0" rpy="0 0 0" />
-      <geometry>
-        <mesh filename="../meshes_new/knee_pitch_r_link.STL" />
+        <mesh filename="package://tiangong3_urdf/meshes/knee_pitch_r_link.STL" />
+      </geometry>
+      <material name="">
+        <color rgba="0.752941176470588 0.752941176470588 0.752941176470588 1" />
+      </material>
+    </visual>
+    <collision>
+      <origin xyz="0 0 0" rpy="0 0 0" />
+      <geometry>
+        <mesh filename="package://tiangong3_urdf/meshes/knee_pitch_r_link.STL" />
       </geometry>
     </collision>
@@ -388,16 +322,16 @@
       <origin xyz="0 0 0" rpy="0 0 0" />
       <geometry>
-        <mesh filename="../meshes_new/ankle_pitch_r_link.STL" />
-      </geometry>
-      <material name="">
-        <color rgba="0.752941176470588 0.752941176470588 0.752941176470588 1" />
-      </material>
-    </visual>
-    <!-- <collision>
-      <origin xyz="0 0 0" rpy="0 0 0" />
-      <geometry>
-        <mesh filename="../meshes_new/ankle_pitch_r_link.STL" />
-      </geometry>
-    </collision> -->
+        <mesh filename="package://tiangong3_urdf/meshes/ankle_pitch_r_link.STL" />
+      </geometry>
+      <material name="">
+        <color rgba="0.752941176470588 0.752941176470588 0.752941176470588 1" />
+      </material>
+    </visual>
+    <collision>
+      <origin xyz="0 0 0" rpy="0 0 0" />
+      <geometry>
+        <mesh filename="package://tiangong3_urdf/meshes/ankle_pitch_r_link.STL" />
+      </geometry>
+    </collision>
   </link>
   <joint name="ankle_pitch_r_joint" type="revolute">
@@ -417,56 +351,14 @@
       <origin xyz="0 0 0" rpy="0 0 0" />
       <geometry>
-        <mesh filename="../meshes_new/ankle_roll_r_link.STL" />
-      </geometry>
-      <material name="">
-        <color rgba="0.752941176470588 0.752941176470588 0.752941176470588 1" />
-      </material>
-    </visual>
-    <!-- <collision>
-      <origin xyz="0 0 0" rpy="0 0 0" />
-      <geometry>
-        <mesh filename="../meshes_new/ankle_roll_r_link.STL" />
-      </geometry>
-    </collision> -->
-    <collision name="foot_right_front_outer">
-      <origin xyz="0.085 -0.03 -0.046" rpy="0 1.5708 0" />
-      <geometry>
-        <cylinder radius="0.012" length="0.06" />
-      </geometry>
-    </collision>
-    <collision name="foot_right_front_inner">
-      <origin xyz="0.085 0.03 -0.046" rpy="0 1.5708 0" />
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