Commit message: Add support for the 29-DoF Tiangong3 robot

File: source/whole_body_tracking/whole_body_tracking/assets/tiangong3/urdf/tiangong3.urdf (robot description, URDF)
Before this commit: robot tiangong3_urdf, 39 links, 38 joints
Joints:
- joint elbow_yaw_l_joint: limit lower=-2.9670597283903604 upper=2.9670597283903604 effort=25.0 velocity=12.217653829810706 -> lower=-2.9670597283903604 upper=2.9670597283903604 effort=40.0 velocity=12.217653829810706
- joint elbow_yaw_r_joint: limit lower=-2.9670597283903604 upper=2.9670597283903604 effort=25.0 velocity=12.217653829810706 -> lower=-2.9670597283903604 upper=2.9670597283903604 effort=40.0 velocity=12.217653829810706
- joint wrist_pitch_l_joint: limit lower=-1.3962634015954636 upper=1.3962634015954636 effort=25.0 velocity=12.217653829810706 -> lower=-1.3962634015954636 upper=1.3962634015954636 effort=40.0 velocity=12.217653829810706
- joint wrist_pitch_r_joint: limit lower=-1.3962634015954636 upper=1.3962634015954636 effort=25.0 velocity=12.217653829810706 -> lower=-1.3962634015954636 upper=1.3962634015954636 effort=40.0 velocity=12.217653829810706
- joint wrist_roll_l_joint: limit lower=-1.3962634015954636 upper=1.3962634015954636 effort=25.0 velocity=12.217653829810706 -> lower=-1.3962634015954636 upper=1.3962634015954636 effort=40.0 velocity=12.217653829810706
- joint wrist_roll_r_joint: limit lower=-1.3962634015954636 upper=1.3962634015954636 effort=25.0 velocity=12.217653829810706 -> lower=-1.3962634015954636 upper=1.3962634015954636 effort=40.0 velocity=12.217653829810706

File: source/whole_body_tracking/whole_body_tracking/assets/tiangong3/urdf/tiangong3.urdf.xacro (robot description, xacro)
@@ -743,5 +743,5 @@
     <child link="elbow_yaw_l_link" />
     <axis xyz="0 0 1" />
-    <limit lower="-2.9670597283903604" upper="2.9670597283903604" effort="25.0" velocity="12.217653829810706" />
+    <limit lower="-2.9670597283903604" upper="2.9670597283903604" effort="40.0" velocity="12.217653829810706" />
   </joint>
   <link name="wrist_pitch_l_link">
@@ -772,5 +772,5 @@
     <child link="wrist_pitch_l_link" />
     <axis xyz="0 1 0" />
-    <limit lower="-1.3962634015954636" upper="1.3962634015954636" effort="25.0" velocity="12.217653829810706" />
+    <limit lower="-1.3962634015954636" upper="1.3962634015954636" effort="40.0" velocity="12.217653829810706" />
   </joint>
   <link name="wrist_roll_l_link">
@@ -801,5 +801,5 @@
     <child link="wrist_roll_l_link" />
     <axis xyz="1 0 0" />
-    <limit lower="-1.3962634015954636" upper="1.3962634015954636" effort="25.0" velocity="12.217653829810706" />
+    <limit lower="-1.3962634015954636" upper="1.3962634015954636" effort="40.0" velocity="12.217653829810706" />
   </joint>
   <link name="left_tcp_link">
@@ -974,5 +974,5 @@
     <child link="elbow_yaw_r_link" />
     <axis xyz="0 0 1" />
-    <limit lower="-2.9670597283903604" upper="2.9670597283903604" effort="25.0" velocity="12.217653829810706" />
+    <limit lower="-2.9670597283903604" upper="2.9670597283903604" effort="40.0" velocity="12.217653829810706" />
   </joint>
   <link name="wrist_pitch_r_link">
@@ -1003,5 +1003,5 @@
     <child link="wrist_pitch_r_link" />
     <axis xyz="0 1 0" />
-    <limit lower="-1.3962634015954636" upper="1.3962634015954636" effort="25.0" velocity="12.217653829810706" />
+    <limit lower="-1.3962634015954636" upper="1.3962634015954636" effort="40.0" velocity="12.217653829810706" />
   </joint>
   <link name="wrist_roll_r_link">
@@ -1032,5 +1032,5 @@
     <child link="wrist_roll_r_link" />
     <axis xyz="1 0 0" />
-    <limit lower="-1.3962634015954636" upper="1.3962634015954636" effort="25.0" velocity="12.217653829810706" />
+    <limit lower="-1.3962634015954636" upper="1.3962634015954636" effort="40.0" velocity="12.217653829810706" />
   </joint>
   <link name="right_tcp_link">

File: source/whole_body_tracking/whole_body_tracking/assets/tiangong3/urdf/tiangong3_29.urdf (robot description, URDF)
Before this commit: robot tiangong3_urdf, 39 links, 38 joints
Joints:
- joint elbow_yaw_l_joint: limit lower=-2.9670597283903604 upper=2.9670597283903604 effort=25.0 velocity=12.217653829810706 -> lower=-2.9670597283903604 upper=2.9670597283903604 effort=40.0 velocity=12.217653829810706
- joint elbow_yaw_r_joint: limit lower=-2.9670597283903604 upper=2.9670597283903604 effort=25.0 velocity=12.217653829810706 -> lower=-2.9670597283903604 upper=2.9670597283903604 effort=40.0 velocity=12.217653829810706
- joint wrist_pitch_l_joint: limit lower=-1.3962634015954636 upper=1.3962634015954636 effort=25.0 velocity=12.217653829810706 -> lower=-1.3962634015954636 upper=1.3962634015954636 effort=40.0 velocity=12.217653829810706
- joint wrist_pitch_r_joint: limit lower=-1.3962634015954636 upper=1.3962634015954636 effort=25.0 velocity=12.217653829810706 -> lower=-1.3962634015954636 upper=1.3962634015954636 effort=40.0 velocity=12.217653829810706
- joint wrist_roll_l_joint: limit lower=-1.3962634015954636 upper=1.3962634015954636 effort=25.0 velocity=12.217653829810706 -> lower=-1.3962634015954636 upper=1.3962634015954636 effort=40.0 velocity=12.217653829810706
- joint wrist_roll_r_joint: limit lower=-1.3962634015954636 upper=1.3962634015954636 effort=25.0 velocity=12.217653829810706 -> lower=-1.3962634015954636 upper=1.3962634015954636 effort=40.0 velocity=12.217653829810706

Commit message: update urdf

File: source/whole_body_tracking/whole_body_tracking/assets/tiangong3/urdf/tiangong3.urdf (robot description, URDF)
Before this commit: robot tiangong3_urdf, 39 links, 38 joints
Links:
- link ankle_pitch_l_link: geometry collision mesh filename=../meshes/ankle_pitch_l_link.STL; visual mesh filename=../meshes/ankle_pitch_l_link.STL
- link ankle_pitch_r_link: geometry collision mesh filename=../meshes/ankle_pitch_r_link.STL; visual mesh filename=../meshes/ankle_pitch_r_link.STL
- link ankle_roll_l_link: geometry collision mesh filename=../meshes/ankle_roll_l_link.STL; visual mesh filename=../meshes/ankle_roll_l_link.STL
- link ankle_roll_r_link: geometry collision mesh filename=../meshes/ankle_roll_r_link.STL; visual mesh filename=../meshes/ankle_roll_r_link.STL
- link camera_body_front_link: geometry collision mesh filename=../meshes/camera_body_front_link.STL; visual mesh filename=../meshes/camera_body_front_link.STL
- link camera_head_link: geometry collision mesh filename=../meshes/camera_head_link.STL; visual mesh filename=../meshes/camera_head_link.STL
- link elbow_pitch_l_link: mass 0.647211 -> 0.780806; geometry collision mesh filename=../meshes/elbow_pitch_l_link.STL; visual mesh filename=../meshes/elbow_pitch_l_link.STL
- link elbow_pitch_r_link: mass 0.647211 -> 0.780806; geometry collision mesh filename=../meshes/elbow_pitch_r_link.STL; visual mesh filename=../meshes/elbow_pitch_r_link.STL
- link elbow_yaw_l_link: mass 0.229689 -> 0.36493; geometry collision mesh filename=../meshes/elbow_yaw_l_link.STL; visual mesh filename=../meshes/elbow_yaw_l_link.STL
- link elbow_yaw_r_link: mass 0.229689 -> 0.36493; geometry collision mesh filename=../meshes/elbow_yaw_r_link.STL; visual mesh filename=../meshes/elbow_yaw_r_link.STL
- link head_pitch_link: mass 0.067829 -> 0.087922; geometry collision mesh filename=../meshes/head_pitch_link.STL; visual mesh filename=../meshes/head_pitch_link.STL
- link head_yaw_link: mass 0.95297 -> 0.968233; geometry collision mesh filename=../meshes/head_yaw_link.STL; visual mesh filename=../meshes/head_yaw_link.STL
- link hip_pitch_l_link: mass 2.221379 -> 2.373121; geometry collision mesh filename=../meshes/hip_pitch_l_link.STL; visual mesh filename=../meshes/hip_pitch_l_link.STL
- link hip_pitch_r_link: mass 2.221379 -> 2.373121; geometry collision mesh filename=../meshes/hip_pitch_r_link.STL; visual mesh filename=../meshes/hip_pitch_r_link.STL
- link hip_roll_l_link: mass 0.560034 -> 0.539594; geometry collision mesh filename=../meshes/hip_roll_l_link.STL; visual mesh filename=../meshes/hip_roll_l_link.STL
- link hip_roll_r_link: mass 0.560034 -> 0.539594; geometry collision mesh filename=../meshes/hip_roll_r_link.STL; visual mesh filename=../meshes/hip_roll_r_link.STL
- link hip_yaw_l_link: mass 5.658158 -> 5.562147; geometry collision mesh filename=../meshes/hip_yaw_l_link.STL; visual mesh filename=../meshes/hip_yaw_l_link.STL
- link hip_yaw_r_link: mass 5.658158 -> 5.562147; geometry collision mesh filename=../meshes/hip_yaw_r_link.STL; visual mesh filename=../meshes/hip_yaw_r_link.STL
- link imu_head_link: geometry collision mesh filename=../meshes/imu_head_link.STL; visual mesh filename=../meshes/imu_head_link.STL
- link imu_waist_link: geometry collision mesh filename=../meshes/imu_waist_link.STL; visual mesh filename=../meshes/imu_waist_link.STL
- link knee_pitch_l_link: mass 3.158584 -> 2.945335; geometry collision mesh filename=../meshes/knee_pitch_l_link.STL; visual mesh filename=../meshes/knee_pitch_l_link.STL
- link knee_pitch_r_link: mass 3.158584 -> 2.945335; geometry collision mesh filename=../meshes/knee_pitch_r_link.STL; visual mesh filename=../meshes/knee_pitch_r_link.STL
- link left_tcp_link: mass 0.457436 -> 0.425076; geometry collision mesh filename=../meshes/left_tcp_link.STL; visual mesh filename=../meshes/left_tcp_link.STL
- link pelvis: mass 10.579253 -> 11.528555; geometry collision mesh filename=../meshes/pelvis.STL; visual mesh filename=../meshes/pelvis.STL
- link radar_head_link: geometry collision mesh filename=../meshes/radar_head_link.STL; visual mesh filename=../meshes/radar_head_link.STL
- link right_tcp_link: mass 0.457436 -> 0.425076; geometry collision mesh filename=../meshes/right_tcp_link.STL; visual mesh filename=../meshes/right_tcp_link.STL
- link shoulder_pitch_l_link: mass 0.914808 -> 0.990828; geometry collision mesh filename=../meshes/shoulder_pitch_l_link.STL; visual mesh filename=../meshes/shoulder_pitch_l_link.STL
- link shoulder_pitch_r_link: mass 0.914808 -> 0.990828; geometry collision mesh filename=../meshes/shoulder_pitch_r_link.STL; visual mesh filename=../meshes/shoulder_pitch_r_link.STL
- link shoulder_roll_l_link: mass 0.319153 -> 0.444503; geometry collision mesh filename=../meshes/shoulder_roll_l_link.STL; visual mesh filename=../meshes/shoulder_roll_l_link.STL
- link shoulder_roll_r_link: mass 0.319153 -> 0.444503; geometry collision mesh filename=../meshes/shoulder_roll_r_link.STL; visual mesh filename=../meshes/shoulder_roll_r_link.STL
- link shoulder_yaw_l_link: mass 1.502215 -> 1.53899; geometry collision mesh filename=../meshes/shoulder_yaw_l_link.STL; visual mesh filename=../meshes/shoulder_yaw_l_link.STL
- link shoulder_yaw_r_link: mass 1.502215 -> 1.53899; geometry collision mesh filename=../meshes/shoulder_yaw_r_link.STL; visual mesh filename=../meshes/shoulder_yaw_r_link.STL
- link waist_pitch_link: mass 10.403447 -> 10.400612; geometry collision mesh filename=../meshes/waist_pitch_link.STL; visual mesh filename=../meshes/waist_pitch_link.STL
- link waist_roll_link: mass 3.595194 -> 3.995987; geometry collision mesh filename=../meshes/waist_roll_link.STL; visual mesh filename=../meshes/waist_roll_link.STL
- link waist_yaw_link: mass 1.688374 -> 1.908803; geometry collision mesh filename=../meshes/waist_yaw_link.STL; visual mesh filename=../meshes/waist_yaw_link.STL
- link wrist_pitch_l_link: mass 0.931823 -> 1.089228; geometry collision mesh filename=../meshes/wrist_pitch_l_link.STL; visual mesh filename=../meshes/wrist_pitch_l_link.STL
- link wrist_pitch_r_link: mass 0.931823 -> 1.089228; geometry collision mesh filename=../meshes/wrist_pitch_r_link.STL; visual mesh filename=../meshes/wrist_pitch_r_link.STL
- link wrist_roll_l_link: mass 0.12 -> 0.154081; geometry collision mesh filename=../meshes/wrist_roll_l_link.STL; visual mesh filename=../meshes/wrist_roll_l_link.STL
- link wrist_roll_r_link: mass 0.12 -> 0.154081; geometry collision mesh filename=../meshes/wrist_roll_r_link.STL; visual mesh filename=../meshes/wrist_roll_r_link.STL
Joints:
- joint ankle_pitch_l_joint: limit lower=-1.2217304763960306 upper=0.5235987755982988 effort=55.0 velocity=14.137166941154069 -> lower=-1.1868238913561442 upper=0.5235987755982988 effort=55.0 velocity=14.137166941154069
- joint ankle_pitch_r_joint: limit lower=-1.2217304763960306 upper=0.5235987755982988 effort=55.0 velocity=14.137166941154069 -> lower=-1.1868238913561442 upper=0.5235987755982988 effort=55.0 velocity=14.137166941154069
- joint camera_head_joint: origin xyz=0.01555 0.011209 -0.00012387 rpy=-1.5659 0 -1.5708 -> xyz=0.01555 0.011078 0 rpy=-1.5708 0 -1.5708
- joint elbow_pitch_l_joint: limit lower=-2.6179938779914944 upper=0.2617993877991494 effort=50.0 velocity=11.455294012539582 -> lower=-2.548180707911721 upper=0.19198621771937624 effort=50.0 velocity=11.455294012539582
- joint elbow_pitch_r_joint: limit lower=-2.6179938779914944 upper=0.2617993877991494 effort=50.0 velocity=11.455294012539582 -> lower=-2.548180707911721 upper=0.19198621771937624 effort=50.0 velocity=11.455294012539582
- joint elbow_yaw_l_joint: limit lower=-2.9670597283903604 upper=2.9670597283903604 effort=40.0 velocity=12.217653829810706 -> lower=-2.844886680750757 upper=2.844886680750757 effort=40.0 velocity=18.325957145940457; origin xyz=-0.02 0 -0.107 rpy=0 0 0 -> xyz=-0.02 0 -0.104 rpy=0 0 0
- joint elbow_yaw_r_joint: limit lower=-2.9670597283903604 upper=2.9670597283903604 effort=40.0 velocity=12.217653829810706 -> lower=-2.844886680750757 upper=2.844886680750757 effort=40.0 velocity=18.325957145940457; origin xyz=-0.02 0 -0.107 rpy=0 0 0 -> xyz=-0.02 0 -0.104 rpy=0 0 0
- joint head_pitch_joint: limit lower=-0.9599310885968813 upper=0.2617993877991494 effort=6.3 velocity=7.644542123735163 -> lower=-0.8726646259971648 upper=0.2617993877991494 effort=6.3 velocity=7.644542123735163; origin xyz=0.0689 -7.7578E-05 -0.0006 rpy=0 0 0 -> xyz=0.0689 -5.5575E-05 -0.0008 rpy=0 0 0
- joint head_yaw_joint: origin xyz=0 0 0.43627 rpy=0 0 0 -> xyz=0.00022262 0 0.43727 rpy=0 0 0
- joint hip_pitch_l_joint: limit lower=-3.141592653589793 upper=2.8797932657906435 effort=235.0 velocity=16.755160819145562 -> lower=-3.0543261909900763 upper=2.792526803190927 effort=235.0 velocity=16.755160819145562
- joint hip_pitch_r_joint: limit lower=-3.141592653589793 upper=2.8797932657906435 effort=235.0 velocity=16.755160819145562 -> lower=-3.0543261909900763 upper=2.792526803190927 effort=235.0 velocity=16.755160819145562
- joint hip_roll_l_joint: origin xyz=9.9595E-05 0.073992 -0.026966 rpy=0.17453 0 0 -> xyz=0 0.073992 -0.026966 rpy=0.17453 0 0
- joint hip_roll_r_joint: origin xyz=9.9595E-05 -0.073992 -0.026966 rpy=-0.17453 0 0 -> xyz=0 -0.073992 -0.026966 rpy=-0.17453 0 0
- joint hip_yaw_l_joint: limit lower=-1.3962634015954636 upper=4.537856055185257 effort=150.0 velocity=13.82300767579509 -> lower=-1.3962634015954636 upper=4.4505895925855405 effort=150.0 velocity=13.82300767579509
- joint hip_yaw_r_joint: limit lower=-4.537856055185257 upper=1.3962634015954636 effort=150.0 velocity=13.82300767579509 -> lower=-4.4505895925855405 upper=1.3962634015954636 effort=150.0 velocity=13.82300767579509
- joint imu_head_joint: origin xyz=-0.057774 0 0.42677 rpy=-3.1416 0 -1.5708 -> xyz=-0.057551 0 0.42777 rpy=-3.1416 0 -1.5708
- joint knee_pitch_l_joint: origin xyz=-0.012927 9.9662E-05 -0.30599 rpy=0 0 0 -> xyz=-0.012927 0 -0.30599 rpy=0 0 0
- joint knee_pitch_r_joint: origin xyz=-0.012927 -9.9662E-05 -0.30599 rpy=0 0 0 -> xyz=-0.012927 0 -0.30599 rpy=0 0 0
- joint left_tcp_joint: origin xyz=0 0 -0.045 rpy=0 0 0 -> xyz=0 0 -0.044 rpy=0 0 0
- joint radar_head_joint: origin xyz=0 0 0.38177 rpy=-3.1416 0 0 -> xyz=0.00022262 0 0.38237 rpy=3.1416 0 1.5708
- joint right_tcp_joint: origin xyz=0 0 -0.045 rpy=0 0 0 -> xyz=0 0 -0.044 rpy=0 0 0
- joint shoulder_pitch_l_joint: limit lower=-2.9670597283903604 upper=2.9670597283903604 effort=90.0 velocity=7.218332720398149 -> lower=-2.844886680750757 upper=2.844886680750757 effort=90.0 velocity=7.218332720398149
- joint shoulder_pitch_r_joint: limit lower=-2.9670597283903604 upper=2.9670597283903604 effort=90.0 velocity=7.218332720398149 -> lower=-2.844886680750757 upper=2.844886680750757 effort=90.0 velocity=7.218332720398149
- joint shoulder_roll_l_joint: limit lower=-0.2617993877991494 upper=3.4033920413889422 effort=90.0 velocity=7.218332720398149 -> lower=-0.19198621771937624 upper=3.3335788713091694 effort=90.0 velocity=7.218332720398149
- joint shoulder_roll_r_joint: limit lower=-3.4033920413889422 upper=0.2617993877991494 effort=90.0 velocity=7.218332720398149 -> lower=-3.3335788713091694 upper=0.19198621771937624 effort=90.0 velocity=7.218332720398149
- joint shoulder_yaw_l_joint: limit lower=-2.9670597283903604 upper=2.9670597283903604 effort=50.0 velocity=11.455294012539582 -> lower=-2.844886680750757 upper=2.844886680750757 effort=50.0 velocity=11.455294012539582
- joint shoulder_yaw_r_joint: limit lower=-2.9670597283903604 upper=2.9670597283903604 effort=50.0 velocity=11.455294012539582 -> lower=-2.844886680750757 upper=2.844886680750757 effort=50.0 velocity=11.455294012539582
- joint waist_pitch_joint: limit lower=-0.5235987755982988 upper=0.9599310885968813 effort=150.0 velocity=13.82300767579509 -> lower=-0.5235987755982988 upper=0.8726646259971648 effort=150.0 velocity=13.82300767579509
- joint waist_roll_joint: origin xyz=0 0 0.0838 rpy=0 0 0 -> xyz=0 0 0.083796 rpy=0 0 0
- joint waist_yaw_joint: limit lower=-2.740166925631097 upper=3.2288591161895095 effort=91.0 velocity=9.42477796076938 -> lower=-2.6179938779914944 upper=3.2288591161895095 effort=91.0 velocity=9.42477796076938
- joint wrist_pitch_l_joint: limit lower=-1.3962634015954636 upper=1.3962634015954636 effort=40.0 velocity=12.217653829810706 -> lower=-1.3264502315156903 upper=1.3264502315156903 effort=40.0 velocity=18.325957145940457; origin xyz=0 0 -0.091 rpy=0 0 0 -> xyz=0 0 -0.0944 rpy=0 0 0
- joint wrist_pitch_r_joint: limit lower=-1.3962634015954636 upper=1.3962634015954636 effort=40.0 velocity=12.217653829810706 -> lower=-1.3264502315156903 upper=1.3264502315156903 effort=40.0 velocity=18.325957145940457; origin xyz=0 0 -0.091 rpy=0 0 0 -> xyz=0 0 -0.0944 rpy=0 0 0
- joint wrist_roll_l_joint: limit lower=-1.3962634015954636 upper=1.3962634015954636 effort=40.0 velocity=12.217653829810706 -> lower=-1.3264502315156903 upper=1.3264502315156903 effort=40.0 velocity=18.325957145940457
- joint wrist_roll_r_joint: limit lower=-1.3962634015954636 upper=1.3962634015954636 effort=40.0 velocity=12.217653829810706 -> lower=-1.3264502315156903 upper=1.3264502315156903 effort=40.0 velocity=18.325957145940457
